File: Hardware/RS-232 Yost DTE.kicad_pcb (KiCad board)
At the start: 2 copper layers, 26 x 50.5 mm, 24 parts, among them J1 Conn_01x06_Female, J2 RJ45, P1 USB_C_Plug_USB2.0, U1 HIN213EIAZ, U2 FT231XS-R

Commit message: Updated files
Centering
Parts:
- added REF**: MountingHole_2.2mm_M2, MountingHole:MountingHole_2.2mm_M2, F.Cu at (140.5, 116.5)
- added REF**: MountingHole_2.2mm_M2, MountingHole:MountingHole_2.2mm_M2, F.Cu at (163.5, 116.5)
- moved P1 0.20 mm to (151.9, 108.1)
Routing:
- net Net-(P1-PadA5): track 5.55 -> 6.31 mm
Other:
- outline, holes or cut-outs redrawn

Commit message: Updates
remember to check orientations
Parts:
- moved J2 7.02 mm to (154.0, 148.5), turned to 180 degrees
Routing:
- net DCD-232: track 34.2 -> 13.5 mm
- net TXD-232: track 27.8 -> 13.4 mm
- net RTS-232: track 21.0 -> 13.2 mm
- net RXD-232: track 23.5 -> 29.9 mm
- net CTS-232: track 33.2 -> 36.4 mm
- net DTR-232: track 25.5 -> 24.0 mm
- net Earth: vias 10 -> 9

Commit message: Updated files
Parts:
- added TP1: TestPoint, TestPoint:TestPoint_Pad_1.5x1.5mm, F.Cu at (146.2, 103.8)
- added TP3: TestPoint, TestPoint:TestPoint_Pad_1.5x1.5mm, F.Cu at (157.6, 103.8)
- P1: footprint SnapEDA Library:GCT_USB4155-03-C_REVA -> Expansion_Card:USB_C_Plug_Molex_105444
- moved P1 3.36 mm to (151.9, 104.8), turned to 0 degrees
Routing:
- net Earth: track 149.2 -> 98.8 mm, vias 9 -> 11
- net Net-(F1-Pad2): track 11.9 -> 18.5 mm, vias 0 -> 2
- net Net-(P1-PadA5): track 6.31 -> 10.4 mm
- net /D+: track 5.04 -> 9.06 mm
- net /D-: track 4.83 -> 8.84 mm
Other:
- board size 26 x 50.5 mm -> 26 x 50.6 mm
