File: Hardware/RS-232 Yost DTE.sch (KiCad schematic (older format))
At the start: 24 parts, among them J1 Conn_01x06_Female, J2 RJ45, P1 USB_C_Plug_USB2.0, U1 HIN213EIAZ, U2 FT231XS-R

Commit message: Updated files
Parts:
- P1: footprint SnapEDA Library:GCT_USB4155-03-C_REVA -> Expansion_Card:USB_C_Plug_Molex_105444
Changed lines of the file:
@@
 F 0 "P1" H 2207 3217 50  0000 C CNN
 F 1 "USB_C_Plug_USB2.0" H 2207 3126 50  0000 C CNN
-F 2 "SnapEDA Library:GCT_USB4155-03-C_REVA" H 2250 2350 50  0001 C CNN
+F 2 "Expansion_Card:USB_C_Plug_Molex_105444" H 2250 2350 50  0001 C CNN
 F 3 "https://www.usb.org/sites/default/files/documents/usb_type-c.zip" H 2250 2350 50  0001 C CNN
 	1    2100 2350
